File: 65c816-sbc-v1/65c816-sbc-v1.kicad_pcb (KiCad board)
At the start: 4 copper layers, 56 parts, among them J1 EXPANSION, J2 SIO, J3 VIA_A, J4 VIA_B, J5 power, SW1 RESET, SW2 NMI, U1 W65C816SxP, U10 W65C22SxP, U11 W65C51NxP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

Commit message: more layout inspired changes
Parts:
- added RN10: 1K, Resistor_THT:R_Array_SIP9, F.Cu at (340.8, 45.3)
- added RN11: 1K, Resistor_THT:R_Array_SIP9, F.Cu at (340.8, 49.6)
- added RN2: 1K, Resistor_THT:R_Array_SIP9, F.Cu at (316.0, 36.6)
- added RN3: 1K, Resistor_THT:R_Array_SIP9, F.Cu at (316.0, 40.9)
- added RN4: 1K, Resistor_THT:R_Array_SIP9, F.Cu at (340.8, 36.6)
- added RN5: 1K, Resistor_THT:R_Array_SIP9, F.Cu at (316.0, 45.3)
- added RN6: 1K, Resistor_THT:R_Array_SIP9, F.Cu at (340.8, 40.9)
- added RN7: 1K, Resistor_THT:R_Array_SIP9, F.Cu at (316.0, 49.6)
- added RN8: 1K, Resistor_THT:R_Array_SIP9, F.Cu at (316.0, 54.0)
- added RN9: 1K, Resistor_THT:R_Array_SIP9, F.Cu at (316.0, 58.3)
- moved J1 109.7 mm to (84.3, 192.0), turned to 90 degrees
- moved C1 98.5 mm to (227.5, -34.7)
- moved C21 98.5 mm to (218.4, -34.7)
- moved C25 98.5 mm to (234.8, -50.8)
- moved C34 98.5 mm to (216.7, -47.0)
- moved C35 98.5 mm to (225.8, -50.8)
- moved C37 98.5 mm to (216.7, -55.1)
- moved D1 98.5 mm to (149.8, -22.9)
- moved D3 98.5 mm to (160.5, -21.0)
- moved J5 98.5 mm to (207.0, -54.6)
- moved R2 98.5 mm to (194.9, -32.8)
- moved U12 98.5 mm to (195.0, -54.8)
- moved U15 98.5 mm to (206.7, -37.5)
- moved C22 98.5 mm to (234.8, -42.7)
- moved C24 98.5 mm to (225.8, -42.7)
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Connections:
- U6 pad 12: BUS_A3 -> BUS_A6
- U6 pad 13: CPU_A6 -> CPU_A5
- U6 pad 14: BUS_A2 -> BUS_A4
- U6 pad 15: CPU_A5 -> CPU_A3
- U6 pad 16: BUS_A1 -> BUS_A2
- U6 pad 17: CPU_A4 -> CPU_A1
- U6 pad 3: BUS_A4 -> BUS_A1
- U6 pad 4: CPU_A1 -> CPU_A2
- U6 pad 5: BUS_A5 -> BUS_A3
- U6 pad 6: CPU_A2 -> CPU_A4
- U6 pad 7: BUS_A6 -> BUS_A5
- U6 pad 8: CPU_A3 -> CPU_A6
- U7 pad 11: CPU_A15 -> CPU_A11
- U7 pad 12: BUS_A11 -> BUS_A12
- U7 pad 13: CPU_A14 -> CPU_A10
- U7 pad 14: BUS_A10 -> BUS_A13
- U7 pad 15: CPU_A13 -> CPU_A9
- U7 pad 16: BUS_A9 -> BUS_A14
- U7 pad 17: CPU_A12 -> CPU_A8
- U7 pad 18: BUS_A8 -> BUS_A15
- U7 pad 2: CPU_A8 -> CPU_A15
- U7 pad 3: BUS_A12 -> BUS_A8
- U7 pad 4: CPU_A9 -> CPU_A14
- U7 pad 5: BUS_A13 -> BUS_A9
- U7 pad 6: CPU_A10 -> CPU_A13
- U7 pad 7: BUS_A14 -> BUS_A10
- U7 pad 8: CPU_A11 -> CPU_A12
- U7 pad 9: BUS_A15 -> BUS_A11
Routing:
- net BUS_DA_LATCH_OE_N: track 0.00 -> 87.4 mm, vias 0 -> 2
- net BUS_A0: track 0.00 -> 61.5 mm, vias 0 -> 1
- net BUS_A15: track 0.00 -> 60.2 mm, vias 0 -> 1
- net BUS_A2: track 0.00 -> 60.0 mm, vias 0 -> 1
- net BUS_A4: track 0.00 -> 58.4 mm, vias 0 -> 1
- net BUS_A6: track 0.00 -> 57.2 mm, vias 0 -> 1
- net BUS_A1: track 0.00 -> 53.8 mm, vias 0 -> 1
- net BUS_A14: track 0.00 -> 53.1 mm, vias 0 -> 1
- net BUS_A3: track 0.00 -> 52.6 mm, vias 0 -> 1
- net BUS_A5: track 0.00 -> 50.8 mm, vias 0 -> 1
- net BUS_A7: track 0.00 -> 49.3 mm, vias 0 -> 1
- net BUS_A13: track 0.00 -> 46.2 mm, vias 0 -> 1
- net CPU_A14: track 0.00 -> 40.5 mm
- net CPU_A15: track 0.00 -> 40.3 mm
- net BUS_A12: track 0.00 -> 39.4 mm, vias 0 -> 1
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
Commit message: update schematic/layout some more; this is quite challenging!
Parts:
- moved J2 159.7 mm to (354.2, 112.9)
- moved J3 149.7 mm to (346.3, 199.9), turned to 180 degrees
- moved U10 127.8 mm to (334.2, 197.6), turned to 180 degrees
- moved J4 124.1 mm to (346.1, 170.9), turned to 180 degrees
- moved J1 68.2 mm to (19.7, 170.2)
- moved U11 59.1 mm to (318.6, 88.1)
- moved U9 8.29 mm to (63.4, 93.3)
- moved U8 8.29 mm to (88.6, 88.1)
- moved U4 1.15 mm to (142.9, 84.5)
Routing:
- net BUS_D2: track 1.92 -> 158.4 mm, vias 0 -> 3
- net BUS_D1: track 1.66 -> 155.9 mm, vias 0 -> 3
- net BUS_D0: track 1.66 -> 153.0 mm, vias 0 -> 3
- net BUS_A13: track 46.2 -> 193.9 mm, vias 1 -> 4
- net BUS_D4: track 1.92 -> 146.6 mm, vias 0 -> 3
- net BUS_D6: track 1.89 -> 145.7 mm, vias 0 -> 3
- net BUS_D5: track 1.89 -> 145.4 mm, vias 0 -> 3
- net BUS_D7: track 0.00 -> 143.2 mm, vias 0 -> 3
- net BUS_A14: track 53.1 -> 185.8 mm, vias 1 -> 4
- net BUS_A15: track 60.2 -> 185.6 mm, vias 1 -> 4
- net BUS_D3: track 1.66 -> 119.8 mm, vias 0 -> 3
- net CPU_VPA: track 0.00 -> 98.9 mm, vias 0 -> 2
- net BUS_A10: track 31.5 -> 121.2 mm, vias 1 -> 2
- net (no net): track 0.00 -> 87.8 mm
- net BUS_A11: track 28.2 -> 115.4 mm, vias 1 -> 2
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
Commit message: another update; i'm not liking how this is working out right now.
Parts:
- C1, C20, C21, C22, C23, C24, C25, C26, C27, C28, C29, C30, C31, C32, C33, C34, C35, C36, C37: footprint Capacitor_THT:C_Rect_L7.5mm_W6.5mm_P5.00mm -> Capacitor_THT:C_Rect_L4.0mm_W2.5mm_P2.50mm
- C3, C38: footprint Capacitor_THT:CP_Radial_D10.0mm_P7.50mm -> Capacitor_THT:CP_Radial_D6.3mm_P2.50mm
- moved C30 268.6 mm to (22.3, 18.2), turned to 90 degrees
- moved X1 252.3 mm to (25.0, 37.7)
- moved C25 221.1 mm to (62.5, 87.8)
- moved J3 214.4 mm to (225.2, 23.1), turned to 270 degrees
- moved J4 210.4 mm to (196.2, 23.3), turned to 270 degrees
- moved U10 195.7 mm to (225.2, 35.1), turned to 270 degrees
- moved C34 194.4 mm to (76.8, 88.0)
- moved U15 191.1 mm to (25.7, 23.8), turned to 90 degrees
- moved C35 176.6 mm to (68.6, 29.8)
- moved C36 166.6 mm to (82.7, 88.0)
- moved C21 160.4 mm to (106.6, 80.3), turned to 90 degrees
- moved J2 157.4 mm to (196.9, 108.0), turned to 270 degrees
- moved C37 150.8 mm to (91.1, 28.3)
- moved C24 141.4 mm to (113.8, 43.7)
- moved C22 126.4 mm to (143.5, 44.7), turned to 90 degrees
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Connections:
- J1 pad 26: BUS_A24 -> CPU_IRQN
- U9 pad 22: BUS_BANK0_OE_N -> BUS_DEV_OE_N
Routing:
- net (no net): track 87.8 -> 0.00 mm
- net BUS_DEV_OE_N: track 0.00 -> 52.5 mm
- net BUS_A1: track 113.1 -> 161.5 mm
- net BUS_A0: track 121.7 -> 169.3 mm
- net BUS_A22: track 26.5 -> 73.4 mm
- net BUS_A21: track 29.5 -> 76.0 mm
- net BUS_A17: track 86.8 -> 132.6 mm
- net BUS_A20: track 33.5 -> 79.2 mm
- net BUS_A19: track 37.5 -> 83.2 mm
- net BUS_A18: track 88.1 -> 133.5 mm
- net BUS_A16: track 109.1 -> 153.8 mm
- net BUS_A3: track 110.3 -> 152.2 mm
- net BUS_A11: track 115.4 -> 156.8 mm, vias 2 -> 3
- net BUS_A2: track 118.4 -> 159.7 mm
- net BUS_A23: track 30.5 -> 70.9 mm
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