File: 65c816-sbc-v1/65c816-sbc-v1.kicad_pcb (KiCad board)
At the start: 4 copper layers, 66 parts, among them J1 EXPANSION, J2 SIO, J3 VIA_A, J4 VIA_B, J5 power, SW1 RESET, SW2 NMI, U1 W65C816SxP, U10 W65C22SxP, U11 W65C51NxP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

Commit message: [65c816] more routing funness
Parts:
- moved U9 216.7 mm to (128.5, 157.6)
- moved U8 187.5 mm to (153.6, 152.4)
- moved U5 40.5 mm to (87.8, 97.1), turned to 270 degrees
- moved J1 33.1 mm to (18.8, 40.4)
- moved U1 33.1 mm to (63.0, 40.3)
- moved U3 33.1 mm to (88.5, 38.4)
- moved U4 33.1 mm to (114.1, 58.6)
- moved U6 33.1 mm to (44.3, 41.1)
- moved U2 33.1 mm to (88.5, 66.1)
- moved U7 33.1 mm to (44.6, 68.9)
Routing:
- net CPU_VDA: track 21.8 -> 78.7 mm
- net BUS_D7: track 6.18 -> 59.4 mm
- net BUS_D6: track 3.06 -> 54.6 mm
- net BUS_D5: track 6.18 -> 56.1 mm
- net CPU_PHI2: track 29.9 -> 79.5 mm
- net BUS_D4: track 3.06 -> 51.3 mm
- net BUS_D3: track 6.18 -> 52.7 mm
- net BUS_D2: track 3.06 -> 48.2 mm
- net CPU_BE: track 31.5 -> 75.7 mm
- net BUS_D1: track 6.18 -> 49.6 mm
- net CPU_RDY: track 31.7 -> 73.7 mm
- net BUS_D0: track 3.06 -> 44.8 mm
- net BUS_A5: track 35.5 -> 73.8 mm, vias 0 -> 1
- net CPU_RW: track 37.8 -> 70.6 mm
- net BUS_A12: track 74.3 -> 100.8 mm
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